File: 00_circuit diagram/briefkastensensor.sch (KiCad schematic (older format))
At the start: 8 parts, among them U1 ATtiny84-20PU, U2 RFM95W

Commit message: beautify circuit diagram
Parts:
- D1: symbol HSDL-9100-021:HSDL-9100-021 -> briefkastensensor-rescue:HSDL-9100-021-HSDL-9100-021
- U1: symbol MCU_Microchip_ATtiny:ATtiny84-20PU -> briefkastensensor-rescue:ATtiny84-20PU-MCU_Microchip_ATtiny
- U2: symbol RF_AM_FM:RFM95W-868S2 -> briefkastensensor-rescue:RFM95W-868S2-RF_AM_FM
Connections:
- net labels added: RX, TX
- wire segments 35 -> 44
Other:
- note added: "HSDL 9100 Proximity Sensor"
- note added: "RFM95W Lora Module"
- note added: "Serial (optional)"
- note added: "Status-LED (optional)"
- moved on the sheet: AE1, D2, R1, R2, R3
