File: 00_circuit_diagram/briefkastensensor.sch (KiCad schematic (older format))
At the start: 8 parts, among them U1 ATtiny84-20PU, U2 RFM95W

Commit message: circuit: add reset button
Parts:
- added SW1: RESET_BUTTON, symbol Switch:SW_Push
Connections:
- wire segments 44 -> 51
Changed lines of the file:
@@
 L power:GND #PWR?
 U 1 1 5CC04235
-P 3650 5350
-F 0 "#PWR?" H 3650 5100 50  0001 C CNN
-F 1 "GND" H 3655 5177 50  0000 C CNN
-F 2 "" H 3650 5350 50  0001 C CNN
-F 3 "" H 3650 5350 50  0001 C CNN
-	1    3650 5350
+P 3200 5375
+F 0 "#PWR?" H 3200 5125 50  0001 C CNN
+F 1 "GND" H 3205 5202 50  0000 C CNN
+F 2 "" H 3200 5375 50  0001 C CNN
+F 3 "" H 3200 5375 50  0001 C CNN
+	1    3200 5375
 	1    0    0    -1
 $EndComp
@@
 Wire Wire Line
 	4650 4700 4250 4700
-Wire Wire Line
-	3650 5200 3650 5350
 Wire Wire Line
 	4450 3250 4450 4200
@@
 Wire Wire Line
 	3650 3350 3650 3400
+Wire Wire Line
+	3650 5200 3650 5300
+Wire Wire Line
+	3650 5300 3475 5300
+Wire Wire Line
+	3200 5300 3200 5375
+$Comp
+L Switch:SW_Push SW1
+U 1 1 602A5F2D
+P 3950 5500
+F 0 "SW1" H 3950 5675 50  0000 C CNN
+F 1 "RESET_BUTTON" H 3950 5400 50  0000 C CNN
+F 2 "" H 3950 5700 50  0001 C CNN
+F 3 "~" H 3950 5700 50  0001 C CNN
+	1    3950 5500
+	1    0    0    -1
+$EndComp
+Wire Wire Line
+	4150 5500 4250 5500
+Wire Wire Line
+	4250 5500 4250 4900
+Wire Wire Line
+	3750 5500 3475 5500
+Connection ~ 3475 5300
+Wire Wire Line
+	3475 5300 3200 5300
+Wire Wire Line
+	3475 5500 3475 5300
 $EndSCHEMATC
